File: kicad/hackpad.kicad_sch (KiCad schematic)
At the start: 44 parts, among them J1 Conn_01x04_MountingPin, U1 MOUDLE-SEEEDUINO-XIAO

Commit message: update kicad
Parts:
- U1: footprint Seeed Studio XIAO Series Library:XIAO-SAMD21-DIP -> Seeed Studio XIAO Series Library:XIAO-RP2040-DIP
Connections:
- no-connect marks 0 -> 2
Changed lines of the file:
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@@
 		(color 0 0 0 0)
 	)
+	(no_connect
+		(at 146.05 67.31)
+	)
+	(no_connect
+		(at 224.79 144.78)
+	)
 	(wire
 		(pts
@@
 	(wire
 		(pts
+			(xy 95.25 49.53) (xy 87.63 49.53)
+		)
+		(stroke
+			(width 0)
+			(type default)
+		)
+	)
+	(wire
+		(pts
+			(xy 100.33 55.88) (xy 97.79 55.88)
+		)
+		(stroke
+			(width 0)
+			(type default)
+		)
+	)
+	(wire
+		(pts
 			(xy 195.58 58.42) (xy 195.58 71.12)
 		)
@@
 	(wire
 		(pts
+			(xy 137.16 50.8) (xy 139.7 50.8)
+		)
+		(stroke
+			(width 0)
+			(type default)
+		)
+	)
+	(wire
+		(pts
 			(xy 140.97 137.16) (xy 156.21 137.16)
 		)
@@
 	(wire
 		(pts
+			(xy 132.08 57.15) (xy 140.97 57.15)
+		)
+		(stroke
+			(width 0)
+			(type default)
+		)
+	)
+	(wire
+		(pts
 			(xy 208.28 58.42) (xy 208.28 71.12)
 		)
@@
 	(wire
 		(pts
+			(xy 139.7 50.8) (xy 139.7 54.61)
+		)
+		(stroke
+			(width 0)
+			(type default)
+		)
+	)
+	(wire
+		(pts
 			(xy 49.53 137.16) (xy 64.77 137.16)
 		)
@@
 	(wire
 		(pts
+			(xy 139.7 54.61) (xy 140.97 54.61)
+		)
+		(stroke
+			(width 0)
+			(type default)
+		)
+	)
+	(wire
+		(pts
 			(xy 171.45 152.4) (xy 186.69 152.4)
 		)
@@
 	(wire
 		(pts
+			(xy 97.79 55.88) (xy 97.79 54.61)
+		)
+		(stroke
+			(width 0)
+			(type default)
+		)
+	)
+	(wire
+		(pts
 			(xy 99.06 85.09) (xy 120.65 85.09)
 		)
@@
 	(wire
 		(pts
+			(xy 97.79 54.61) (xy 87.63 54.61)
+		)
+		(stroke
+			(width 0)
+			(type default)
+		)
+	)
+	(wire
+		(pts
 			(xy 125.73 137.16) (xy 140.97 137.16)
 		)
@@
 	(wire
 		(pts
+			(xy 104.14 52.07) (xy 87.63 52.07)
+		)
+		(stroke
+			(width 0)
+			(type default)
+		)
+	)
+	(wire
+		(pts
 			(xy 208.28 30.48) (xy 208.28 33.02)
 		)
@@
 	(symbol
 		(lib_id "power:+3.3V")
-		(at 140.97 57.15 90)
+		(at 132.08 57.15 0)
 		(unit 1)
 		(exclude_from_sim no)
@@
 		(fields_autoplaced yes)
 		(property "Reference" "#PWR07"
-			(at 144.78 57.15 0)
+			(at 132.08 60.96 0)
 			(effects
 				(font
@@
 		)
 		(property "Value" "+3.3V"
-			(at 137.16 57.1499 90)
+			(at 132.08 52.07 0)
 			(effects
 				(font
 					(size 1.27 1.27)
 				)
-				(justify left)
 			)
 		)
 		(property "Footprint" ""
-			(at 140.97 57.15 0)
+			(at 132.08 57.15 0)
 			(effects
 				(font
@@
 		)
 		(property "Datasheet" ""
-			(at 140.97 57.15 0)
+			(at 132.08 57.15 0)
 			(effects
 				(font
@@
 		)
 		(property "Description" "Power symbol creates a global label with name \"+3.3V\""
-			(at 140.97 57.15 0)
+			(at 132.08 57.15 0)
 			(effects
 				(font
@@
 	(symbol
 		(lib_id "power:GND")
-		(at 140.97 54.61 270)
+		(at 137.16 50.8 0)
 		(unit 1)
 		(exclude_from_sim no)
@@
 		(fields_autoplaced yes)
 		(property "Reference" "#PWR06"
-			(at 134.62 54.61 0)
+			(at 137.16 57.15 0)
 			(effects
 				(font
@@
 		)
 		(property "Value" "GND"
-			(at 137.16 54.6099 90)
+			(at 137.16 55.88 0)
 			(effects
 				(font
 					(size 1.27 1.27)
 				)
-				(justify right)
 			)
 		)
 		(property "Footprint" ""
-			(at 140.97 54.61 0)
+			(at 137.16 50.8 0)
 			(effects
 				(font
@@
 		)
 		(property "Datasheet" ""
-			(at 140.97 54.61 0)
+			(at 137.16 50.8 0)
 			(effects
 				(font
@@
 		)
 		(property "Description" "Power symbol creates a global label with name \"GND\" , ground"
-			(at 140.97 54.61 0)
+			(at 137.16 50.8 0)
 			(effects
 				(font
@@
 	(symbol
 		(lib_id "power:+3.3V")
-		(at 87.63 54.61 270)
+		(at 100.33 55.88 0)
 		(unit 1)
 		(exclude_from_sim no)
@@
 		(fields_autoplaced yes)
 		(property "Reference" "#PWR01"
-			(at 83.82 54.61 0)
+			(at 100.33 59.69 0)
 			(effects
 				(font
@@
 		)
 		(property "Value" "+3.3V"
-			(at 91.44 54.6099 90)
+			(at 100.33 50.8 0)
 			(effects
 				(font
 					(size 1.27 1.27)
 				)
-				(justify left)
 			)
 		)
 		(property "Footprint" ""
-			(at 87.63 54.61 0)
+			(at 100.33 55.88 0)
 			(effects
 				(font
@@
 		)
 		(property "Datasheet" ""
-			(at 87.63 54.61 0)
+			(at 100.33 55.88 0)
 			(effects
 				(font
@@
 		)
 		(property "Description" "Power symbol creates a global label with name \"+3.3V\""
-			(at 87.63 54.61 0)
+			(at 100.33 55.88 0)
 			(effects
 				(font
@@
 	(symbol
 		(lib_id "power:GND")
-		(at 87.63 52.07 90)
+		(at 104.14 52.07 0)
 		(unit 1)
 		(exclude_from_sim no)
@@
 		(fields_autoplaced yes)
 		(property "Reference" "#PWR02"
-			(at 93.98 52.07 0)
+			(at 104.14 58.42 0)
 			(effects
 				(font
@@
 		)
 		(property "Value" "GND"
-			(at 91.44 52.0699 90)
+			(at 104.14 57.15 0)
 			(effects
 				(font
 					(size 1.27 1.27)
 				)
-				(justify right)
 			)
 		)
 		(property "Footprint" ""
-			(at 87.63 52.07 0)
+			(at 104.14 52.07 0)
 			(effects
 				(font
@@
 		)
 		(property "Datasheet" ""
-			(at 87.63 52.07 0)
+			(at 104.14 52.07 0)
 			(effects
 				(font
@@
 		)
 		(property "Description" "Power symbol creates a global label with name \"GND\" , ground"
-			(at 87.63 52.07 0)
+			(at 104.14 52.07 0)
 			(effects
 				(font
@@
 	(symbol
 		(lib_id "power:+5V")
-		(at 87.63 49.53 270)
+		(at 95.25 49.53 0)
 		(unit 1)
 		(exclude_from_sim no)
@@
 		(fields_autoplaced yes)
 		(property "Reference" "#PWR03"
-			(at 83.82 49.53 0)
+			(at 95.25 53.34 0)
 			(effects
 				(font
@@
 		)
 		(property "Value" "+5V"
-			(at 91.44 49.5299 90)
+			(at 95.25 44.45 0)
 			(effects
 				(font
 					(size 1.27 1.27)
 				)
-				(justify left)
 			)
 		)
 		(property "Footprint" ""
-			(at 87.63 49.53 0)
+			(at 95.25 49.53 0)
 			(effects
 				(font
@@
 		)
 		(property "Datasheet" ""
-			(at 87.63 49.53 0)
+			(at 95.25 49.53 0)
 			(effects
 				(font
@@
 		)
 		(property "Description" "Power symbol creates a global label with name \"+5V\""
-			(at 87.63 49.53 0)
+			(at 95.25 49.53 0)
 			(effects
 				(font
@@
 			)
 		)
-		(property "Footprint" "Seeed Studio XIAO Series Library:XIAO-SAMD21-DIP"
+		(property "Footprint" "Seeed Studio XIAO Series Library:XIAO-RP2040-DIP"
 			(at 49.53 54.61 0)
 			(effects
